File: 4bitCounter/schematic.kicad_pcb (KiCad board)
At the start: 2 copper layers, 20 parts, among them J2 Conn_01x02_Pin, Q1 PN2222A, U1 NE555P, U3 74LS161

Commit message: Update footprints and pcb
Parts:
- Q1: footprint CounterProject:transistor -> CounterProject:Transistor
- R4: footprint 4bitCounter:Resistor -> CounterProject:Resistor
- U1: footprint Package_DIP:DIP-8_W7.62mm -> CounterProject:Timer; moved to F.Cu
- U3: footprint Package_DIP:DIP-16_W7.62mm -> CounterProject:CounterChip; moved to F.Cu
- moved J2 89.0 mm to (233.2, 148.9), turned to -90 degrees
- moved U1 78.3 mm to (228.9, 143.9)
- moved R3 71.8 mm to (262.0, 114.0), turned to 180 degrees
- moved R4 66.3 mm to (251.4, 119.2), turned to -90 degrees
- moved D1 64.0 mm to (208.4, 89.5), turned to 0 degrees
- moved R2 53.7 mm to (218.7, 137.2), turned to -90 degrees
- moved D2 48.2 mm to (216.9, 89.7), turned to 0 degrees
- moved C3 47.7 mm to (254.2, 134.2), turned to -90 degrees
- moved C2 45.6 mm to (261.2, 122.9), turned to -90 degrees
- moved R5 42.0 mm to (243.9, 116.5), turned to 90 degrees
- moved R7 39.5 mm to (203.0, 112.0), turned to 180 degrees
- moved Q1 37.7 mm to (240.2, 123.7), turned to -90 degrees
- moved C1 33.3 mm to (218.4, 129.9), turned to 90 degrees
- moved D3 31.8 mm to (225.7, 89.7), turned to 0 degrees
- moved R8 29.1 mm to (207.7, 106.5), turned to 90 degrees
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Routing:
- net Net-(U1-DIS): track 182.0 -> 73.4 mm
- net Net-(D1-K): track 293.0 -> 230.6 mm
- net Net-(U1-THR): track 99.1 -> 52.5 mm
- net Net-(U1-CV): track 41.2 -> 18.5 mm
- net Net-(C2-Pad1): track 40.2 -> 18.4 mm
- net Net-(D1-A): track 10.5 -> 27.9 mm
- net Net-(Q1-B): track 27.8 -> 12.1 mm
- net Net-(J2-Pin_1): track 149.3 -> 161.0 mm
- net Net-(Q1-E): track 27.8 -> 17.1 mm
- net Net-(D3-A): track 7.90 -> 18.4 mm
- net Net-(U3-Q1): track 13.8 -> 23.8 mm
- net Net-(U3-Q2): track 6.26 -> 16.2 mm
- net Net-(D4-A): track 12.8 -> 19.5 mm
- net Net-(U3-Q3): track 6.01 -> 12.1 mm
- net Net-(D2-A): track 12.0 -> 16.6 mm
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Other:
- board outline added: 96.1 x 81.3 mm

Commit message: Update pcb schematic
Parts:
- moved R3 51.6 mm to (210.8, 120.7), turned to 0 degrees
- moved C2 42.2 mm to (219.1, 120.7), turned to 0 degrees
- moved R4 35.6 mm to (215.9, 117.5), turned to 180 degrees
- moved J2 31.5 mm to (234.3, 117.5), turned to 0 degrees
- moved Q1 29.2 mm to (214.0, 110.8), turned to 180 degrees
- moved R5 24.9 mm to (219.1, 117.5), turned to 0 degrees
- moved U1 23.3 mm to (227.2, 120.7), turned to -90 degrees
- moved R7 20.2 mm to (219.1, 99.7), turned to 90 degrees
- moved U3 19.6 mm to (219.0, 114.2), turned to 0 degrees
- moved R8 18.4 mm to (224.8, 99.7)
- moved C3 17.9 mm to (238.8, 125.1), turned to 90 degrees
- moved R1 17.4 mm to (215.9, 106.7), turned to 90 degrees
- moved R9 17.3 mm to (230.5, 99.7)
- moved R10 16.7 mm to (236.2, 99.7)
- moved C1 12.8 mm to (231.1, 131.4), turned to 0 degrees
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Routing:
- net Net-(U1-DIS): track 73.4 -> 177.9 mm
- net Net-(J2-Pin_1): track 161.0 -> 101.2 mm
- net Net-(D1-K): track 230.6 -> 176.1 mm
- net Net-(U1-THR): track 52.5 -> 27.6 mm
- net Net-(D1-A): track 27.9 -> 4.44 mm
- net Net-(U3-Q0): track 27.3 -> 9.14 mm
- net Net-(U3-Q1): track 23.8 -> 7.82 mm
- net Net-(D4-A): track 19.5 -> 4.38 mm
- net Net-(D3-A): track 18.4 -> 4.44 mm
- net Net-(U1-CV): track 18.5 -> 5.55 mm
- net Net-(D2-A): track 16.6 -> 4.45 mm
- net Net-(C2-Pad1): track 18.4 -> 6.36 mm
- net Net-(U3-Q2): track 16.2 -> 7.56 mm
- net Net-(Q1-B): track 12.1 -> 6.93 mm
- net Net-(Q1-E): track 17.1 -> 12.2 mm
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
Commit message: Update pcb routing
Parts:
- moved R7 3.06 mm to (219.3, 102.7)
- moved D1 3.06 mm to (216.8, 93.2)
- moved D2 3.06 mm to (222.5, 93.2)
- moved D3 3.06 mm to (228.2, 93.2)
- moved D4 3.06 mm to (233.9, 93.3)
- moved R10 3.06 mm to (236.5, 102.7)
- moved R8 3.06 mm to (225.0, 102.7)
- moved R9 3.06 mm to (230.8, 102.7)
- moved C2 0.38 mm to (219.1, 121.0)
Routing:
- net Net-(U1-DIS): track 177.9 -> 119.1 mm
- net Net-(D1-K): track 176.1 -> 143.5 mm
- net Net-(J2-Pin_1): track 101.2 -> 84.8 mm
- net Net-(U3-Q1): track 7.82 -> 4.67 mm
- net Net-(U3-Q2): track 7.56 -> 4.62 mm
- net Net-(U3-Q0): track 9.14 -> 6.48 mm
- net Net-(U3-Q3): track 8.88 -> 7.03 mm
- net Net-(Q1-E): track 12.2 -> 11.5 mm
- net Net-(U1-THR): track 27.6 -> 26.9 mm

Commit message: update pcb and schematic
Parts:
- moved D1 14.4 mm to (224.1, 105.7)
- moved D2 14.4 mm to (229.8, 105.7)
- moved D3 14.4 mm to (235.5, 105.7)
- moved D4 14.4 mm to (241.2, 105.7)
- moved R10 14.4 mm to (243.8, 115.2)
- moved R8 14.4 mm to (232.3, 115.2)
- moved R9 14.4 mm to (238.1, 115.2)
- moved R7 14.4 mm to (226.6, 115.2)
- moved C3 14.3 mm to (245.9, 137.5)
- moved R5 14.3 mm to (226.2, 129.9)
- moved C1 14.3 mm to (238.3, 143.9)
- moved J2 14.3 mm to (241.4, 129.9)
- moved R4 14.3 mm to (223.0, 129.9)
- moved Q1 14.3 mm to (221.1, 123.2)
- moved R1 14.3 mm to (223.0, 119.1)
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Connections:
- net Net-(D1-K) renamed GND
Routing:
- net GND: track 143.5 -> 138.6 mm
- net Net-(U1-DIS): track 119.1 -> 117.4 mm
- net Net-(J2-Pin_1): track 84.8 -> 83.2 mm
