File: ergo20411/ergo20411.kicad_pcb (KiCad board)
At the start: 2 copper layers, 22 parts, among them J1 Conn_01x02_Pin, U1 LM555xN, U2 4017

Commit message: Update pcb
Parts:
- moved D7 34.6 mm to (143.5, 78.4)
- moved J1 30.7 mm to (157.0, 90.5)
- moved D9 27.3 mm to (151.3, 81.7)
- moved R1 26.8 mm to (190.4, 90.1), turned to -90 degrees
- moved D8 26.6 mm to (151.5, 84.7), turned to -90 degrees
- moved R2 24.1 mm to (182.8, 83.5), turned to -90 degrees
- moved C3 18.8 mm to (179.9, 77.0)
- moved C1 17.3 mm to (167.5, 91.4), turned to 90 degrees
- moved R3 15.4 mm to (174.4, 72.1)
- moved R5 15.3 mm to (151.5, 71.1), turned to -90 degrees
- moved C2 14.2 mm to (162.3, 94.7), turned to 90 degrees
- moved R7 12.1 mm to (169.6, 71.8), turned to -90 degrees
- moved U1 9.18 mm to (172.6, 87.9), turned to -90 degrees
- moved R6 7.68 mm to (160.7, 83.3), turned to 180 degrees
- moved D6 3.17 mm to (160.6, 79.5)
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Routing:
- net Net-(U1-THR): track 0.00 -> 66.4 mm
- net Net-(J1-Pin_1): track 0.00 -> 41.7 mm
- net GND: track 15.1 -> 42.3 mm
- net Net-(U1-CV): track 0.00 -> 19.5 mm
- net Net-(U2-Reset): track 33.7 -> 14.4 mm
- net Net-(D9-A): track 0.00 -> 19.3 mm
- net Net-(U1-Q): track 0.00 -> 17.1 mm
- net Net-(D1-K): track 52.2 -> 38.1 mm
- net Net-(U2-Cout): track 17.0 -> 4.00 mm
- net Net-(U1-DIS): track 0.00 -> 11.6 mm
- net Net-(D7-A): track 0.00 -> 8.11 mm
- net Net-(D8-A): track 0.00 -> 5.78 mm
- net Net-(U2-CLK): track 0.00 -> 4.38 mm
- net Net-(D6-A): track 8.46 -> 5.64 mm
- net Net-(D5-K): track 9.60 -> 8.44 mm
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